File: crown-layout.brd (EAGLE design)
At the start: 302 x 51.5 mm, 21 parts

Commit message: Just cleanup stuff
Parts:
- U$1: value SMDUINODIS-CONNECTED-PINS -> SMDUINO; device pcb_crown:SMDUINO -> SMDuino:SMDUINO
- moved POWER_ON 25.1 mm to (10.2, 37.8), turned to 180 degrees
- moved ALWAYS_ON 23.8 mm to (8.92, 39.0)
- moved A7 19.2 mm to (32.4, 61.4), turned to 0 degrees
- moved D2 18.4 mm to (32.4, 55.0), turned to 0 degrees
- moved SKIP-PTH1 9.99 mm to (17.5, 61.0), turned to 90 degrees
- moved C4 7.73 mm to (17.8, 55.1), turned to 90 degrees
- moved C3 7.37 mm to (40.4, 54.9), turned to 90 degrees
- moved A6 7.25 mm to (32.4, 68.4), turned to 0 degrees
- moved U$1 4.06 mm to (17.8, 26.4)
Connections:
- net N$16 renamed PD7
- net N$17 renamed PD6
- removed net N$14: U$1.A0
- removed net N$15: U$1.A1
- removed net N$18: U$1.PD5
- removed net N$19: U$1.PD4
- removed net N$2 (its old number): A7.P$1, A7.P$2, U$1.A7
- removed net N$20: U$1.PD3
- removed net N$6: A6.P$1, A6.P$2, U$1.A6
- removed net N$7 (its old number): U$1.A5
- removed net N$8: U$1.A4
- removed net N$9: D2.P$1, D2.P$2, U$1.PD2
- removed net PTH-DI: PTH-END-NODE.1, U$1.PB3, U$2.P$26, U$2.P$7
- removed net SMD-DI: SMD-END-NODE.1, U$1.PB2, U$2.P$24, U$2.P$5
- new net A0: U$1.A0, U$2.P$13
- new net A1: U$1.A1, U$2.P$14
- new net A2: U$1.A2, U$2.P$15
- new net A3: A6.P$1, A6.P$2, U$1.A3
- new net A4: U$1.A4, U$2.P$31
- new net A5: U$1.A5, U$2.P$32
- new net A6: A7.P$1, A7.P$2, U$1.A6
- new net A7: D2.P$1, D2.P$2, U$1.A7
- new net N$24: U$1.AREF
- new net PB0: SMD-END-NODE.1, U$1.PB0, U$2.P$24, U$2.P$5
- new net PB1: PTH-END-NODE.1, U$1.PB1, U$2.P$26, U$2.P$7
- new net PB2: U$1.PB2, U$2.P$9
- new net PB3: U$1.PB3, U$2.P$10
- new net PB4: U$1.PB4, U$2.P$11
- new net PB5: U$2.P$12
- new net PD2: U$1.PD2
- new net PD3: U$1.PD3, U$2.P$30
- new net PD4: U$1.PD4, U$2.P$29
- new net PD5: U$1.PD5, U$2.P$28
- net GND: now also U$2.P$18, U$2.P$37
- net N$4: now also U$2.P$19
- net PTH-DO: now also U$2.P$38
- net RXI: now also U$2.P$34
- net TXO: now also U$2.P$33
- net VBAT: now also POWER_ON.1, U$2.P$16, U$2.P$35; no longer POWER_ON.5
- net VLIVE: now also U$2.P$17, U$2.P$36
Routing:
- net PTH-DI: track 98.6 -> 0.00 mm
- net SMD-DI: track 93.2 -> 0.00 mm
- net PB0: track 0.00 -> 92.2 mm
- net PB1: track 0.00 -> 85.5 mm
- net VBAT: track 163.0 -> 204.8 mm
- net A4: track 0.00 -> 40.3 mm
- net N$9: track 38.7 -> 0.00 mm
- net N$2 (its old number): track 37.5 -> 0.00 mm
- net A5: track 0.00 -> 37.0 mm
- net VLIVE: track 238.7 -> 205.4 mm
- net A2: track 0.00 -> 30.6 mm
- net A3: track 0.00 -> 28.3 mm
- net RXI: track 0.00 -> 25.5 mm
- net A1: track 0.00 -> 23.9 mm
- net PB2: track 0.00 -> 22.0 mm
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- added copper zone on layer 1, net GND
Other:
- board size 302 x 51.5 mm -> 57.8 x 51.5 mm
- board text removed: "PB2"
- board text removed: "PB3"
