File: crown-face.sch (EAGLE design)
At the start: 21 parts

Commit message: Fixed it! :D
Parts:
- U$1: value SMDUINODIS-CONNECTED-PINS -> SMDUINO; device pcb_crown:SMDUINODIS-CONNECTED-PINS -> SMDuino:SMDUINO
Connections:
- net N$16 renamed PD7
- net N$17 renamed PD6
- removed net N$14: U$1.A0
- removed net N$15: U$1.A1
- removed net N$18: U$1.PD5
- removed net N$19: U$1.PD4
- removed net N$2 (its old number): A7.P$1, U$1.A7
- removed net N$20: U$1.PD3
- removed net N$6: A6.P$1, U$1.A6
- removed net N$7 (its old number): U$1.A5
- removed net N$8: U$1.A4
- removed net N$9: D2.P$1, U$1.PD2
- removed net PTH-DI: PTH-END-NODE.1, U$1.PB3, U$2.P$26, U$2.P$7
- removed net SMD-DI: SMD-END-NODE.1, U$1.PB2, U$2.P$24, U$2.P$5
- new net A0: U$1.A0, U$2.P$13
- new net A1: U$1.A1, U$2.P$14
- new net A2: U$1.A2, U$2.P$15
- new net A3: A6.P$1, U$1.A3
- new net A4: U$1.A4, U$2.P$31
- new net A5: U$1.A5, U$2.P$32
- new net A6: A7.P$1, U$1.A6
- new net A7: D2.P$1, U$1.A7
- new net N$24: U$1.AREF
- new net PB0: SMD-END-NODE.1, U$1.PB0, U$2.P$24, U$2.P$5
- new net PB1: PTH-END-NODE.1, U$1.PB1, U$2.P$26, U$2.P$7
- new net PB2: U$1.PB2, U$2.P$9
- new net PB3: U$1.PB3, U$2.P$10
- new net PB4: U$1.PB4, U$2.P$11
- new net PB5: U$2.P$12
- new net PD2: U$1.PD2
- new net PD3: U$1.PD3, U$2.P$30
- new net PD4: U$1.PD4, U$2.P$29
- new net PD5: U$1.PD5, U$2.P$28
- net GND: now also U$2.P$18, U$2.P$37
- net N$4: now also U$2.P$19
- net PTH-DO: now also U$2.P$38
- net RXI: now also U$2.P$34
- net TXO: now also U$2.P$33
- net VBAT: now also POWER_ON.1, U$2.P$16, U$2.P$35; no longer POWER_ON.5
- net VLIVE: now also U$2.P$17, U$2.P$36

Commit message: Just cleanup stuff
Parts:
- added JMP1, JMP2, JMP3, JMP4, JMP5, JMP6, JMP7: SOLDERJUMPERNC2, SparkFun-Passives:SOLDERJUMPERNC2
Connections:
- removed net N$2: U$1.PB5
- net A0: now also JMP3.2
- net A1: now also JMP2.2
- net A2: now also JMP1.2
- net A4: now also JMP4.1
- net A5: now also JMP3.1
- net PB2: now also JMP7.2
- net PB3: now also JMP6.2
- net PB4: now also JMP5.2
- net PB5: now also JMP4.2, U$1.PB5
- net PD3: now also JMP5.1
- net PD4: now also JMP6.1
- net PD5: now also JMP7.1
- net RXI: now also JMP1.1
- net TXO: now also JMP2.1
Changed lines of the file:
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@@
 <part name="ALWAYS_ON" library="SparkFun-Passives" deviceset="SOLDERJUMPER" device="NC2" value=""/>
 <part name="U$1" library="SMDuino" deviceset="SMDUINO" device=""/>
+<part name="JMP1" library="SparkFun-Passives" deviceset="SOLDERJUMPER" device="NC2" value=""/>
+<part name="JMP2" library="SparkFun-Passives" deviceset="SOLDERJUMPER" device="NC2" value=""/>
+<part name="JMP3" library="SparkFun-Passives" deviceset="SOLDERJUMPER" device="NC2" value=""/>
+<part name="JMP4" library="SparkFun-Passives" deviceset="SOLDERJUMPER" device="NC2" value=""/>
+<part name="JMP5" library="SparkFun-Passives" deviceset="SOLDERJUMPER" device="NC2" value=""/>
+<part name="JMP6" library="SparkFun-Passives" deviceset="SOLDERJUMPER" device="NC2" value=""/>
+<part name="JMP7" library="SparkFun-Passives" deviceset="SOLDERJUMPER" device="NC2" value=""/>
 </parts>
 <sheets>
@@
 <instance part="ALWAYS_ON" gate="1" x="-2.54" y="99.06" rot="R180"/>
 <instance part="U$1" gate="G$1" x="-66.04" y="40.64"/>
+<instance part="JMP1" gate="1" x="91.44" y="73.66"/>
+<instance part="JMP2" gate="1" x="91.44" y="68.58"/>
+<instance part="JMP3" gate="1" x="91.44" y="63.5"/>
+<instance part="JMP4" gate="1" x="91.44" y="58.42"/>
+<instance part="JMP5" gate="1" x="91.44" y="53.34"/>
+<instance part="JMP6" gate="1" x="91.44" y="48.26"/>
+<instance part="JMP7" gate="1" x="91.44" y="43.18"/>
 </instances>
 <busses>
@@
 <wire x1="48.26" y1="71.12" x2="33.02" y2="71.12" width="0.2032" layer="91"/>
 <label x="33.02" y="71.12" size="1.778" layer="95"/>
+<pinref part="JMP1" gate="1" pin="1"/>
+<wire x1="86.36" y1="73.66" x2="76.2" y2="73.66" width="0.2032" layer="91"/>
+<label x="78.74" y="73.66" size="1.778" layer="95"/>
+<wire x1="48.26" y1="71.12" x2="73.66" y2="71.12" width="0.2032" layer="91"/>
+<wire x1="73.66" y1="71.12" x2="76.2" y2="73.66" width="0.2032" layer="91"/>
 </segment>
 </net>
@@
 <wire x1="48.26" y1="66.04" x2="33.02" y2="66.04" width="0.2032" layer="91"/>
 <label x="33.02" y="66.04" size="1.778" layer="95"/>
+<pinref part="JMP2" gate="1" pin="1"/>
+<wire x1="86.36" y1="68.58" x2="76.2" y2="68.58" width="0.2032" layer="91"/>
+<label x="78.74" y="68.58" size="1.778" layer="95"/>
+<wire x1="48.26" y1="66.04" x2="73.66" y2="66.04" width="0.2032" layer="91"/>
+<wire x1="73.66" y1="66.04" x2="76.2" y2="68.58" width="0.2032" layer="91"/>
 </segment>
 </net>
@@
 <pinref part="U$2" gate="G$1" pin="P$32"/>
 <label x="33.02" y="60.96" size="1.778" layer="95"/>
+<pinref part="JMP3" gate="1" pin="1"/>
+<wire x1="86.36" y1="63.5" x2="76.2" y2="63.5" width="0.2032" layer="91"/>
+<label x="78.74" y="63.5" size="1.778" layer="95"/>
+<wire x1="48.26" y1="60.96" x2="73.66" y2="60.96" width="0.2032" layer="91"/>
+<wire x1="73.66" y1="60.96" x2="76.2" y2="63.5" width="0.2032" layer="91"/>
 </segment>
 </net>
@@
 <pinref part="U$2" gate="G$1" pin="P$31"/>
 <label x="33.02" y="55.88" size="1.778" layer="95"/>
+<pinref part="JMP4" gate="1" pin="1"/>
+<wire x1="86.36" y1="58.42" x2="78.74" y2="58.42" width="0.2032" layer="91"/>
+<label x="78.74" y="58.42" size="1.778" layer="95"/>
+<wire x1="48.26" y1="55.88" x2="76.2" y2="55.88" width="0.2032" layer="91"/>
+<wire x1="76.2" y1="55.88" x2="78.74" y2="58.42" width="0.2032" layer="91"/>
 </segment>
 </net>
@@
 <wire x1="139.7" y1="60.96" x2="149.86" y2="60.96" width="0.2032" layer="91"/>
 <label x="147.32" y="60.96" size="1.778" layer="95"/>
+<pinref part="JMP3" gate="1" pin="2"/>
+<wire x1="96.52" y1="63.5" x2="104.14" y2="63.5" width="0.2032" layer="91"/>
+<label x="101.6" y="63.5" size="1.778" layer="95"/>
+<wire x1="104.14" y1="63.5" x2="106.68" y2="60.96" width="0.2032" layer="91"/>
+<wire x1="106.68" y1="60.96" x2="139.7" y2="60.96" width="0.2032" layer="91"/>
 </segment>
 </net>
@@
 <wire x1="139.7" y1="66.04" x2="149.86" y2="66.04" width="0.2032" layer="91"/>
 <label x="147.32" y="66.04" size="1.778" layer="95"/>
+<pinref part="JMP2" gate="1" pin="2"/>
+<wire x1="96.52" y1="68.58" x2="104.14" y2="68.58" width="0.2032" layer="91"/>
+<label x="101.6" y="68.58" size="1.778" layer="95"/>
+<wire x1="104.14" y1="68.58" x2="106.68" y2="66.04" width="0.2032" layer="91"/>
+<wire x1="106.68" y1="66.04" x2="139.7" y2="66.04" width="0.2032" layer="91"/>
 </segment>
 </net>
@@
 <label x="33.02" y="40.64" size="1.778" layer="95"/>
 <pinref part="U$2" gate="G$1" pin="P$28"/>
+<pinref part="JMP7" gate="1" pin="1"/>
+<wire x1="86.36" y1="43.18" x2="81.28" y2="43.18" width="0.2032" layer="91"/>
+<label x="78.74" y="43.18" size="1.778" layer="95"/>
+<wire x1="48.26" y1="40.64" x2="78.74" y2="40.64" width="0.2032" layer="91"/>
+<wire x1="78.74" y1="40.64" x2="81.28" y2="43.18" width="0.2032" layer="91"/>
 </segment>
 </net>
@@
 <label x="33.02" y="45.72" size="1.778" layer="95"/>
 <pinref part="U$2" gate="G$1" pin="P$29"/>
+<pinref part="JMP6" gate="1" pin="1"/>
+<wire x1="86.36" y1="48.26" x2="81.28" y2="48.26" width="0.2032" layer="91"/>
+<label x="78.74" y="48.26" size="1.778" layer="95"/>
+<wire x1="48.26" y1="45.72" x2="78.74" y2="45.72" width="0.2032" layer="91"/>
+<wire x1="78.74" y1="45.72" x2="81.28" y2="48.26" width="0.2032" layer="91"/>
 </segment>
 </net>
@@
 <label x="33.02" y="50.8" size="1.778" layer="95"/>
 <pinref part="U$2" gate="G$1" pin="P$30"/>
+<pinref part="JMP5" gate="1" pin="1"/>
+<wire x1="86.36" y1="53.34" x2="81.28" y2="53.34" width="0.2032" layer="91"/>
+<label x="78.74" y="53.34" size="1.778" layer="95"/>
+<wire x1="48.26" y1="50.8" x2="78.74" y2="50.8" width="0.2032" layer="91"/>
+<wire x1="78.74" y1="50.8" x2="81.28" y2="53.34" width="0.2032" layer="91"/>
 </segment>
 </net>
@@
 <wire x1="139.7" y1="71.12" x2="154.94" y2="71.12" width="0.2032" layer="91"/>
 <label x="147.32" y="71.12" size="1.778" layer="95"/>
+<pinref part="JMP1" gate="1" pin="2"/>
+<wire x1="96.52" y1="73.66" x2="104.14" y2="73.66" width="0.2032" layer="91"/>
+<label x="101.6" y="73.66" size="1.778" layer="95"/>
+<wire x1="104.14" y1="73.66" x2="106.68" y2="71.12" width="0.2032" layer="91"/>
+<wire x1="106.68" y1="71.12" x2="139.7" y2="71.12" width="0.2032" layer="91"/>
 </segment>
 </net>
@@
 <wire x1="-81.28" y1="53.34" x2="-78.74" y2="53.34" width="0.2032" layer="91"/>
 <wire x1="-78.74" y1="53.34" x2="-78.74" y2="30.48" width="0.2032" layer="91"/>
+<label x="-76.2" y="53.34" size="1.778" layer="95"/>
 </segment>
 </net>
@@
 <wire x1="-48.26" y1="38.1" x2="-48.26" y2="35.56" width="0.2032" layer="91"/>
 <pinref part="U$1" gate="G$1" pin="GND2"/>
-</segment>
-</net>
-<net name="N$2" class="0">
-<segment>
-<wire x1="-50.8" y1="38.1" x2="-50.8" y2="35.56" width="0.2032" layer="91"/>
-<pinref part="U$1" gate="G$1" pin="PB5"/>
 </segment>
 </net>
@@
 <wire x1="139.7" y1="55.88" x2="149.86" y2="55.88" width="0.2032" layer="91"/>
 <label x="147.32" y="55.88" size="1.778" layer="95"/>
+<pinref part="JMP4" gate="1" pin="2"/>
+<wire x1="96.52" y1="58.42" x2="104.14" y2="58.42" width="0.2032" layer="91"/>
+<label x="101.6" y="58.42" size="1.778" layer="95"/>
+<wire x1="104.14" y1="58.42" x2="106.68" y2="55.88" width="0.2032" layer="91"/>
+<wire x1="106.68" y1="55.88" x2="139.7" y2="55.88" width="0.2032" layer="91"/>
+</segment>
+<segment>
+<wire x1="-50.8" y1="38.1" x2="-50.8" y2="35.56" width="0.2032" layer="91"/>
+<pinref part="U$1" gate="G$1" pin="PB5"/>
 </segment>
 </net>
@@
 <wire x1="144.78" y1="43.18" x2="149.86" y2="43.18" width="0.2032" layer="91"/>
 <label x="147.32" y="43.18" size="1.778" layer="95"/>
+<pinref part="JMP7" gate="1" pin="2"/>
+<wire x1="96.52" y1="43.18" x2="104.14" y2="43.18" width="0.2032" layer="91"/>
+<label x="101.6" y="43.18" size="1.778" layer="95"/>
+<wire x1="104.14" y1="43.18" x2="106.68" y2="40.64" width="0.2032" layer="91"/>
+<wire x1="106.68" y1="40.64" x2="139.7" y2="40.64" width="0.2032" layer="91"/>
 </segment>
 </net>
@@
 <wire x1="139.7" y1="45.72" x2="149.86" y2="45.72" width="0.2032" layer="91"/>
 <label x="147.32" y="45.72" size="1.778" layer="95"/>
+<pinref part="JMP6" gate="1" pin="2"/>
+<wire x1="96.52" y1="48.26" x2="104.14" y2="48.26" width="0.2032" layer="91"/>
+<label x="101.6" y="48.26" size="1.778" layer="95"/>
+<wire x1="139.7" y1="45.72" x2="106.68" y2="45.72" width="0.2032" layer="91"/>
+<wire x1="106.68" y1="45.72" x2="104.14" y2="48.26" width="0.2032" layer="91"/>
 </segment>
 </net>
@@
 <wire x1="-68.58" y1="55.88" x2="-81.28" y2="55.88" width="0.2032" layer="91"/>
 <wire x1="-83.82" y1="53.34" x2="-81.28" y2="55.88" width="0.2032" layer="91"/>
+<label x="-76.2" y="55.88" size="1.778" layer="95"/>
 </segment>
 </net>
@@
 <wire x1="139.7" y1="50.8" x2="149.86" y2="50.8" width="0.2032" layer="91"/>
 <label x="147.32" y="50.8" size="1.778" layer="95"/>
-</segment>
-</net>
+<pinref part="JMP5" gate="1" pin="2"/>
+<wire x1="96.52" y1="53.34" x2="104.14" y2="53.34" width="0.2032" layer="91"/>
+<label x="101.6" y="53.34" size="1.778" layer="95"/>
+<wire x1="104.14" y1="53.34" x2="106.68" y2="50.8" width="0.2032" layer="91"/>
+<wire x1="106.68" y1="50.8" x2="139.7" y2="50.8" width="0.2032" layer="91"/>
+</segment>
+</net>

Commit message: forgot a connection on skip-smd bits
Connections:
- net N$10: now also SKIP-SMD2.2
Changed lines of the file:
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@@
 <pinref part="SMD2" gate="G$1" pin="DIN"/>
 <wire x1="218.44" y1="63.5" x2="200.66" y2="71.12" width="0.2032" layer="91"/>
+<pinref part="SKIP-SMD2" gate="1" pin="2"/>
+<wire x1="195.58" y1="53.34" x2="195.58" y2="66.04" width="0.2032" layer="91"/>
+<wire x1="195.58" y1="66.04" x2="200.66" y2="71.12" width="0.2032" layer="91"/>
 </segment>
 </net>
