File: crown-F.brd (EAGLE design)
At the start: 57.8 x 50.8 mm, 97 parts

Commit message: forgot a connection on skip-smd bits
Connections:
- net N$10: now also SKIP-SMD2.2
Routing:
- net N$10: track 28.2 -> 33.2 mm, vias 1 -> 2
Changed lines of the file:
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@@
 <contactref element="C3" pad="2"/>
 <contactref element="C4" pad="2"/>
-<wire x1="13.462" y1="7.62" x2="21.082" y2="7.62" width="0" layer="19" extent="1-16"/>
 <wire x1="21.082" y1="7.62" x2="31.75" y2="7.62" width="1.27" layer="1"/>
 <wire x1="31.75" y1="7.62" x2="39.116" y2="7.62" width="1.27" layer="1"/>
-<wire x1="39.116" y1="7.62" x2="46.482" y2="7.62" width="0" layer="19" extent="1-16"/>
 <wire x1="39.116" y1="7.62" x2="56.4642" y2="7.62" width="1.27" layer="1"/>
 <wire x1="22.516" y1="14.91" x2="21.26" y2="14.91" width="0.254" layer="1"/>
@@
 <wire x1="39.116" y1="12.192" x2="39.116" y2="8.89" width="0.254" layer="16"/>
 <wire x1="39" y1="12.192" x2="39.116" y2="12.192" width="0.254" layer="16"/>
-<wire x1="46.482" y1="8.89" x2="46.482" y2="7.62" width="0" layer="19" extent="1-16"/>
 <via x="39.116" y="8.89" extent="1-16" drill="0.3302"/>
 <wire x1="39.116" y1="8.89" x2="39.116" y2="7.62" width="0.254" layer="1"/>
 <via x="21.082" y="8.89" extent="1-16" drill="0.3302"/>
 <wire x1="21.082" y1="8.89" x2="21.082" y2="7.62" width="0.254" layer="1"/>
-<wire x1="13.462" y1="8.89" x2="13.462" y2="7.62" width="0" layer="19" extent="1-16"/>
 <via x="31.75" y="8.89" extent="1-16" drill="0.3048"/>
 <wire x1="31.75" y1="8.89" x2="31.75" y2="7.62" width="0.508" layer="1"/>
@@
 <contactref element="C1" pad="1"/>
 <contactref element="C2" pad="1"/>
-<wire x1="11.684" y1="10.16" x2="19.05" y2="10.16" width="0" layer="19" extent="1-16"/>
 <wire x1="19.05" y1="10.16" x2="26.67" y2="10.16" width="1.143" layer="1"/>
 <wire x1="26.67" y1="10.16" x2="29.21" y2="10.16" width="1.143" layer="1"/>
 <wire x1="29.21" y1="10.16" x2="37.1856" y2="10.16" width="1.143" layer="1"/>
-<wire x1="37.1856" y1="10.16" x2="44.45" y2="10.16" width="0" layer="19" extent="1-16"/>
 <wire x1="37.1856" y1="10.16" x2="56.5912" y2="10.16" width="1.143" layer="1"/>
-<wire x1="11.684" y1="8.89" x2="11.684" y2="10.16" width="0" layer="19" extent="1-16"/>
 <wire x1="19.166" y1="12.192" x2="19.166" y2="8.89" width="0.2032" layer="16"/>
 <wire x1="19.166" y1="8.89" x2="19.05" y2="8.89" width="0.2032" layer="16"/>
@@
 <via x="29.21" y="8.89" extent="1-16" drill="0.3048"/>
 <wire x1="29.21" y1="8.89" x2="29.21" y2="10.16" width="0.508" layer="1"/>
-<wire x1="44.45" y1="8.89" x2="44.45" y2="10.16" width="0" layer="19" extent="1-16"/>
 <contactref element="U$2" pad="P$17"/>
 <wire x1="0.254" y1="43.18" x2="6.096" y2="43.18" width="0.508" layer="16"/>
@@
 <wire x1="36.576" y1="17.018" x2="38.1" y2="17.018" width="0.2032" layer="1"/>
 <wire x1="38.1" y1="17.018" x2="39.192" y2="18.11" width="0.2032" layer="1"/>
-<wire x1="39.192" y1="18.11" x2="40.55" y2="18.11" width="0.2032" layer="1"/>
+<wire x1="39.192" y1="18.11" x2="39.37" y2="18.11" width="0.2032" layer="1"/>
+<wire x1="39.37" y1="18.11" x2="40.55" y2="18.11" width="0.2032" layer="1"/>
 <wire x1="24.892" y1="16.3631" x2="24.7849" y2="16.256" width="0.2032" layer="16"/>
 <wire x1="24.7849" y1="16.256" x2="21.336" y2="16.256" width="0.2032" layer="16"/>
 <wire x1="21.336" y1="16.256" x2="21.082" y2="16.002" width="0.2032" layer="16"/>
 <via x="21.082" y="16.002" extent="1-16" drill="0.3048"/>
+<contactref element="SKIP-SMD2" pad="2"/>
+<wire x1="43.18" y1="16.9227" x2="39.4653" y2="16.9227" width="0.2032" layer="16"/>
+<wire x1="39.4653" y1="16.9227" x2="39.37" y2="17.018" width="0.2032" layer="16"/>
+<via x="39.37" y="17.018" extent="1-16" drill="0.3048"/>
+<wire x1="39.37" y1="17.018" x2="39.37" y2="18.11" width="0.2032" layer="1"/>
 </signal>
 <signal name="A0">

Commit message: fixed incorrect resistor value
Other:
- board text added: "PIXEL LINE TERMINATION (500 OHM RES)"
- board text removed: "PIXEL LINE TERMINATION (150 OHM RES)"
Changed lines of the file:
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@@
 <text x="12.954" y="16.51" size="0.762" layer="22" font="vector" ratio="15" rot="MR90" align="bottom-center">PIXEL LINE
 TERMINATION
-(150 OHM RES)</text>
+(500 OHM RES)</text>
 <text x="4.572" y="7.62" size="0.762" layer="22" font="vector" ratio="15" rot="MR0" align="center-right">GND</text>
 <text x="4.572" y="5.08" size="0.762" layer="22" font="vector" ratio="15" rot="MR0" align="center-right">VBAT</text>
