File: negativecircuit.brd (EAGLE design)
At the start: 6 parts

Commit message: Prep final project files for publication
Parts:
- removed E$2, E$3, E$4: (no value), SparkFun-Passives:AXIAL-0.3EZ
- removed E$7: (no value), SparkFun-LED:LED5MM
- added C1, R1, R2, R3: (no value), SparkFun-Passives:AXIAL-0.3EZ
- added LED: (no value), SparkFun-LED:LED5MM
- renumbered E$1 to 555
Connections:
- removed net S$3: E$7.A
- new net S$10: R2.P$2
- new net S$9: 555.1, LED.A, R1.P$1, R1.P$2
- net S$2: now also LED.K; no longer E$7.K
- net S$8: now also 555.8
Routing:
- net S$9: track 0.00 -> 72.1 mm
- net S$3: track 20.3 -> 0.00 mm
- net S$6: track 35.6 -> 27.2 mm
- net S$8: track 48.3 -> 42.9 mm
- net S$10: track 0.00 -> 5.08 mm
- net S$4: track 22.9 -> 25.4 mm
- net S$2: track 8.89 -> 6.60 mm
- net S$7: track 2.54 -> 1.78 mm
- net S$5: track 2.54 -> 1.78 mm
- net S$1: track 2.54 -> 1.78 mm
Other:
- board text removed: "555"
